Commit message: new package tm5_700_grip_description

File: src/robotiq/robotiq_description/urdf/robotiq_85_gripper.transmission.xacro (robot description, xacro)
@@ -5,5 +5,5 @@
       <type>transmission_interface/SimpleTransmission</type>
       <joint name="${prefix}robotiq_85_left_knuckle_joint">
-        <hardwareInterface>PositionJointInterface</hardwareInterface>
+        <hardwareInterface>EffortJointInterface</hardwareInterface>
         <!-- <hardwareInterface>EffortJointInterface</hardwareInterface> -->
       </joint>

File: src/tmr_ros1/tm_description/urdf/tm.transmission.xacro (robot description, xacro)
@@ -1,9 +1,9 @@
 <?xml version="1.0"?>
 <robot xmlns:xacro="http://www.ros.org/wiki/xacro">
-  <xacro:macro name="tm_arm_transmission" params="prefix">
+  <xacro:macro name="tm_arm_transmission" params="prefix hw_interface">
     <transmission name="${prefix}shoulder_1_trans">
       <type>transmission_interface/SimpleTransmission</type>
       <joint name="${prefix}shoulder_1_joint">
-        <hardwareInterface>hardware_interface/PositionJointInterface</hardwareInterface>
+        <hardwareInterface>${hw_interface}</hardwareInterface>
       </joint>
       <actuator name="${prefix}shoulder_1_motor">
@@ -14,5 +14,5 @@
       <type>transmission_interface/SimpleTransmission</type>
       <joint name="${prefix}shoulder_2_joint">
-        <hardwareInterface>hardware_interface/PositionJointInterface</hardwareInterface>
+        <hardwareInterface>${hw_interface}</hardwareInterface>
       </joint>
       <actuator name="${prefix}shoulder_2_motor">
@@ -23,5 +23,5 @@
       <type>transmission_interface/SimpleTransmission</type>
       <joint name="${prefix}elbow_1_joint">
-        <hardwareInterface>hardware_interface/PositionJointInterface</hardwareInterface>
+        <hardwareInterface>${hw_interface}</hardwareInterface>
       </joint>
       <actuator name="${prefix}elbow_1_motor">
@@ -32,5 +32,5 @@
       <type>transmission_interface/SimpleTransmission</type>
       <joint name="${prefix}wrist_1_joint">
-        <hardwareInterface>hardware_interface/PositionJointInterface</hardwareInterface>
+        <hardwareInterface>${hw_interface}</hardwareInterface>
       </joint>
       <actuator name="${prefix}wrist_1_motor">
@@ -41,5 +41,5 @@
       <type>transmission_interface/SimpleTransmission</type>
       <joint name="${prefix}wrist_2_joint">
-        <hardwareInterface>hardware_interface/PositionJointInterface</hardwareInterface>
+        <hardwareInterface>${hw_interface}</hardwareInterface>
       </joint>
       <actuator name="${prefix}wrist_2_motor">
@@ -50,5 +50,5 @@
       <type>transmission_interface/SimpleTransmission</type>
       <joint name="${prefix}wrist_3_joint">
-        <hardwareInterface>hardware_interface/PositionJointInterface</hardwareInterface>
+        <hardwareInterface>${hw_interface}</hardwareInterface>
       </joint>
       <actuator name="${prefix}wrist_3_motor">

File: src/tmr_ros1/tm_description/urdf/tm700.urdf.xacro (robot description, xacro)
@@ -2,48 +2,19 @@
 <robot name="tm700" xmlns:xacro="http://www.ros.org/wiki/xacro">
   <!-- transmission -->
-  <xacro:include filename="$(find tm_description)/urdf/tm.transmission.xacro" />
-  <!-- Mass parameters -->
-  <property name="pi" value="3.14159265" />
-  <property name="base_mass" value="1.0" />
-  <property name="shoulder_mass" value="4.5" />
-  <property name="arm_1_mass" value="10.5" />
-  <property name="arm_2_mass" value="2.1" />
-  <property name="wrist_1_mass" value="1.45" />
-  <property name="wrist_2_mass" value="1.45" />
-  <property name="wrist_3_mass" value="0.4" />
-  <!-- Kinematic model -->
-  <!-- Properties from tmcontrol.conf -->
-  <!--
-    DH for TM700:
-    a = [0.00000, 0.329, 0.3115,  0.00000,  0.00000,  0.0000]
-    d = [0.1451,  0.00000,  0.00000,  -0.1222,  0.106,  0.1144]
-    alpha = [ -1.570796327, 0, 0, 1.570796327, 1.570796327, 0 ]
-    q_home_offset = [0, -1.570796327, 0, 1.570796327, 0, 0]
-    joint_direction = [-1, -1, 1, -1, 1, 1]
-    mass = [4.5, 10.5, 2.1, 1.45, 1.45, 0.4]
-    center_of_mass = [ [0, -0.02561, 0.00193], [0.2125, 0, 0.11336], [0.11993, 0.0, 0.0265], [0, -0.0018, 0.01634], [0, 0.0018,0.01634], [0, 0, -0.001159] ](tm700)
-  -->
-  <property name="tm_d1" value="0.1451" />
-  <property name="tm_a2" value="0.3290" />
-  <property name="tm_a3" value="0.3115" />
-  <property name="tm_d4" value="0.1222" />
-  <property name="tm_d5" value="0.1060" />
-  <property name="tm_d6" value="0.1144" />
-  <!-- offsets for shoulder/elbow joints -->
-  <property name="shoulder_offset" value="-0.146" />  <!-- measured from model -->
-  <property name="elbow_offset" value="0.1298" /> <!-- measured from model -->
-  <property name="wrist_offset" value="${-tm_d4 - elbow_offset - shoulder_offset}" />
-  <!-- link lengths used in model -->
-  <property name="shoulder_height" value="${tm_d1}" />
-  <property name="arm_1_length" value="${tm_a2}" />
-  <property name="arm_2_length" value="${tm_a3}" />
-  <property name="wrist_1_length" value="tm_d5}" />
-  <property name="wrist_2_length" value="${tm_d5}" />
-  <property name="wrist_3_length" value="0.0565" />
-  <property name="ee_length" value="${tm_d6 - wrist_3_length}" />
-  <xacro:macro name="cylinder_inertial" params="radius length mass *origin">
+  <xacro:include filename="$(find tm5_description)/urdf/tm.transmission.xacro" />
+  <xacro:include filename="$(find tm5_description)/urdf/tm.gazebo.xacro" />
+    <xacro:macro name="cylinder_inertial_y" params="radius length mass *origin">
     <inertial>
       <mass value="${mass}" />
-      <insert_block name="origin" />
+      <xacro:insert_block name="origin" />
+      <inertia ixx="${0.0833333 * mass * (3 * radius * radius + length * length)}" ixy="0.0" ixz="0.0"
+        iyy="${0.5 * mass * radius * radius}" iyz="0.0"
+        izz="${0.0833333 * mass * (3 * radius * radius + length * length)}" />
+    </inertial>
+  </xacro:macro>
+  <xacro:macro name="cylinder_inertial_z" params="radius length mass *origin">
+    <inertial>
+      <mass value="${mass}" />
+      <xacro:insert_block name="origin" />
       <inertia ixx="${0.0833333 * mass * (3 * radius * radius + length * length)}" ixy="0.0" ixz="0.0"
         iyy="${0.0833333 * mass * (3 * radius * radius + length * length)}" iyz="0.0"
@@ -51,238 +22,306 @@
     </inertial>
   </xacro:macro>
-  <xacro:macro name="tm700_robot" params="prefix joint_limited">
-    <!-- transmission prefix -->
-    <xacro:tm_arm_transmission prefix="${prefix}" />
+  <xacro:macro name="tm5_700_robot" params="prefix joint_limited stl_mesh
+    shoulder_1_lower_limit:=${-1.5*pi}    shoulder_1_upper_limit:=${1.5*pi}
+    shoulder_2_lower_limit:=${-pi}    shoulder_2_upper_limit:=${pi}
+    elbow_lower_limit:=${-pi}    elbow_upper_limit:=${pi}
+    wrist_1_lower_limit:=${-pi}    wrist_1_upper_limit:=${pi}
+    wrist_2_lower_limit:=${-pi}    wrist_2_upper_limit:=${pi}
+    wrist_3_lower_limit:=${-1.5*pi}    wrist_3_upper_limit:=${1.5*pi}
+    transmission_hw_interface:=hardware_interface/PositionJointInterface
+    safety_limits:=false safety_pos_margin:=0.15
+    safety_k_position:=20">
+    <!-- Inertia parameters -->
+    <xacro:property name="base_mass" value="1.0" />
+    <xacro:property name="shoulder_mass" value="4.5" />
+    <xacro:property name="arm_1_mass" value="11.0" />
+    <xacro:property name="arm_2_mass" value="2.5" />
+    <xacro:property name="wrist_1_mass" value="1.45" />
+    <xacro:property name="wrist_2_mass" value="1.45" />
+    <xacro:property name="wrist_3_mass" value="0.4" />
+    <!-- Kinematic model -->
+    <!-- Properties from tmcontrol.conf -->
+    <!--
+      DH for TM5-700:
+      a = [0.0000, 0.3290, 0.3115,  0.0000,  0.0000,  0.0000]
+      d = [0.1452,  0.0000,  0.0000,  -0.1223,  0.1060,  0.11315]
+      alpha = [-0.5*pi, 0, 0, 0.5*pi, 0.5*pi, 0]
+      q_home_offset = [0, -0.5*pi, 0, 0.5*pi, 0, 0]
+      joint_direction = [-1, -1, 1, -1, 1, 1]
+      mass = [4.5, 10.5, 2.1, 1.45, 1.45, 0.4]
+      center_of_mass = [ [0, -0.02561, 0.00193], [0.2125, 0, 0.11336], [0.11993, 0.0, 0.0265], [0, -0.0018, 0.01634], [0, 0.0018,0.01634], [0, 0, -0.001159] ](tm900)
+    -->
+    <xacro:property name="tm_d1" value="0.1452" />
+    <xacro:property name="tm_a2" value="0.3290" />
+    <xacro:property name="tm_a3" value="0.3115" />
+    <xacro:property name="tm_d4" value="0.1223" />
+    <xacro:property name="tm_d5" value="0.1060" />
+    <xacro:property name="tm_d6" value="0.11315" />
+    <!-- offsets for shoulder/elbow joints -->
+    <xacro:property name="wrist_offset" value="${tm_d5}" />
+    <xacro:property name="shoulder_offset" value="0.146" />
+    <xacro:property name="elbow_offset" value="${wrist_offset + shoulder_offset - tm_d4}" /> <!-- 0.1297 -->
+    <!-- link lengths -->
+    <xacro:property name="shoulder_height" value="${tm_d1}" />
+    <xacro:property name="arm_1_length" value="${tm_a2}" />
+    <xacro:property name="arm_2_length" value="${tm_a3}" />
+    <!-- <xacro:property name="wrist_1_length" value="${tm_d5}" /> -->
+    <xacro:property name="wrist_2_length" value="${tm_d5}" />
+    <xacro:property name="wrist_3_length" value="${tm_d6}" />
+    <!--xacro:property name="ee_length" value="${tm_d6 - wrist_3_length}" /-->
+    <xacro:property name="shoulder_radius" value="0.060" />
+    <xacro:property name="arm_1_radius" value="0.060" />
+    <xacro:property name="elbow_radius" value="0.060" />
+    <xacro:property name="arm_2_radius" value="0.045" />
+    <xacro:property name="wrist_radius" value="0.045" />
+    <xacro:tm_arm_transmission prefix="${prefix}" hw_interface="${transmission_hw_interface}" />
+    <xacro:tm_arm_gazebo prefix="${prefix}" />
     <link name="${prefix}base_link" >
       <visual>
         <geometry>
-	  <mesh filename="package://tm_description/meshes/tm700/visual/Base.STL" />
-        </geometry>
-        <material name="Grey">
-          <color rgba="0.5 0.5 0.5 1.0"/>
-        </material>
-      </visual>
-      <collision>
-        <geometry>
-	  <mesh filename="package://tm_description/meshes/tm700/collision/base.STL" />
-        </geometry>
-      </collision>
-      <xacro:cylinder_inertial radius="0.06" length="0.05" mass="${base_mass}">
-        <origin xyz="0.0 0.0 0.0" rpy="0 0 0" />
-      </xacro:cylinder_inertial>
-    </link>
-    <link name="${prefix}shoulder_1_link">
-      <visual>
-        <geometry>
-	  <mesh filename="package://tm_description/meshes/tm700/visual/Shoulder1.STL" />
-        </geometry>
-        <material name="DarkOlive">
-          <color rgba="0.3 0.3 0.25 1.0"/>
-        </material>
-      </visual>
-      <collision>
-        <geometry>
-	  <mesh filename="package://tm_description/meshes/tm700/collision/shoulder_1.STL" />
-        </geometry>
-      </collision>
-      <xacro:cylinder_inertial radius="0.06" length="0.15" mass="${shoulder_mass}">
-        <origin xyz="0.0 0.0 0.0" rpy="0 0 0" />
-      </xacro:cylinder_inertial>
+        <xacro:unless value="${stl_mesh}">
+          <mesh filename="package://tm5_description/meshes/tm5_900/visual/tm5_base.obj" />
+        </xacro:unless>
+        <xacro:if value="${stl_mesh}">
+          <mesh filename="package://tm5_description/meshes/tm5_900/visual/tm5_base.stl" />
+        </xacro:if>
+        </geometry>
+        <material name="LightGrey">
+          <color rgba="0.5 0.5 0.5 1.0" />
+        </material>
+      </visual>
+      <collision>
+        <geometry>
+          <mesh filename="package://tm5_description/meshes/tm5_900/collision/tm5_base_c.stl" />
+        </geometry>
+      </collision>
+      <xacro:cylinder_inertial_y radius="0.06" length="0.05" mass="${base_mass}">
+        <origin xyz="0 0 0" rpy="0 0 0" />
+      </xacro:cylinder_inertial_y>
     </link>
     <joint name="${prefix}shoulder_1_joint" type="revolute">
       <parent link="${prefix}base_link" />
       <child link = "${prefix}shoulder_1_link" />
-      <origin xyz="0.0 0.0 ${shoulder_height}" rpy="${-0.5 * pi} 0.0 0.0" />
-      <axis xyz="0 -1 0" />
-      <xacro:unless value="${joint_limited}">
-        <limit lower="${-2.0 * pi}" upper="${2.0 * pi}" effort="150.0" velocity="3.15"/>
-      </xacro:unless>
-      <xacro:if value="${joint_limited}">
-        <limit lower="${-pi}" upper="${pi}" effort="150.0" velocity="3.15"/>
-      </xacro:if>
-      <dynamics damping="0.0" friction="0.0"/>
-    </joint>
-    <link name="${prefix}arm_1_link">
-      <visual>
-        <geometry>
-	  <mesh filename="package://tm_description/meshes/tm700/visual/Arm1.STL" />
-        </geometry>
-        <material name="DarkOlive">
-          <color rgba="0.3 0.3 0.25 1.0"/>
-        </material>
-      </visual>
-      <collision>
-        <geometry>
-	  <mesh filename="package://tm_description/meshes/tm700/collision/arm_1.STL" />
-        </geometry>
-      </collision>
-      <xacro:cylinder_inertial radius="0.06" length="0.56" mass="${arm_1_mass}">
-        <origin xyz="0.0 0.0 0.28" rpy="0 0 0" />
-      </xacro:cylinder_inertial>
+      <origin xyz="0 ${shoulder_height} 0" rpy="0 0 0" />
+      <axis xyz="0 1 0" />
+      <limit lower="${shoulder_1_lower_limit}" upper="${shoulder_1_upper_limit}" effort="150.0" velocity="3.15" />
+      <xacro:if value="${safety_limits}">
+        <safety_controller soft_lower_limit="${shoulder_1_lower_limit + safety_pos_margin}" soft_upper_limit="${shoulder_1_upper_limit - safety_pos_margin}" k_position="${safety_k_position}" k_velocity="0.0" />
+      </xacro:if>
+      <dynamics damping="0.0" friction="0.0" />
+    </joint>
+    <link name="${prefix}shoulder_1_link">
+      <visual>
+        <geometry>
+        <xacro:unless value="${stl_mesh}">
+          <mesh filename="package://tm5_description/meshes/tm5_900/visual/tm_400w_01.obj" />
+        </xacro:unless>
+        <xacro:if value="${stl_mesh}">
+          <mesh filename="package://tm5_description/meshes/tm5_900/visual/tm_400w_01.stl" />
+        </xacro:if>
+        </geometry>
+        <material name="DarkOlive">
+          <color rgba="0.3 0.3 0.25 1.0" />
+        </material>
+      </visual>
+      <collision>
+        <geometry>
+          <mesh filename="package://tm5_description/meshes/tm5_900/collision/tm_400w_01_c.stl" />
+        </geometry>
+      </collision>
+      <xacro:cylinder_inertial_y radius="0.06" length="0.15" mass="${shoulder_mass}">
+        <origin xyz="0 0 0" rpy="0 0 0" />
+      </xacro:cylinder_inertial_y>
     </link>
     <joint name="${prefix}shoulder_2_joint" type="revolute">
       <parent link="${prefix}shoulder_1_link" />
       <child link = "${prefix}arm_1_link" />
-      <origin xyz="0.0 0.0 ${shoulder_offset}" rpy="0.0 0.0 ${-0.5 * pi}" />
-      <axis xyz="0 0 1" />
-      <xacro:unless value="${joint_limited}">
-        <limit lower="${-1.5 * pi}" upper="${1.5 * pi}" effort="150.0" velocity="3.15"/>
-      </xacro:unless>
-      <xacro:if value="${joint_limited}">
-        <limit lower="${-pi}" upper="${pi}" effort="150.0" velocity="3.15"/>
-      </xacro:if>
-      <dynamics damping="0.0" friction="0.0"/>
-    </joint>
-    <link name="${prefix}arm_2_link">
-      <visual>
-        <geometry>
-	  <mesh filename="package://tm_description/meshes/tm700/visual/Arm2.STL" />
-        </geometry>
-        <material name="DarkOlive">
-          <color rgba="0.3 0.3 0.25 1.0"/>
-        </material>
-      </visual>
-      <collision>
-        <geometry>
-	  <mesh filename="package://tm_description/meshes/tm700/collision/arm_2.STL" />
-        </geometry>
-      </collision>
-      <xacro:cylinder_inertial radius="0.06" length="0.5" mass="${arm_2_mass}">
-        <origin xyz="0.0 0.0 0.25" rpy="0 0 0" />
-      </xacro:cylinder_inertial>
-    </link>
-    <joint name="${prefix}elbow_1_joint" type="revolute">
+      <origin xyz="0 0 ${shoulder_offset}" rpy="0 0 0" />
+      <axis xyz="0 0 -1" />
+      <limit lower="${shoulder_2_lower_limit}" upper="${shoulder_2_upper_limit}" effort="150.0" velocity="3.15" />
+      <xacro:if value="${safety_limits}">
+        <safety_controller soft_lower_limit="${shoulder_2_lower_limit + safety_pos_margin}" soft_upper_limit="${shoulder_2_upper_limit - safety_pos_margin}" k_position="${safety_k_position}" k_velocity="0.0" />
+      </xacro:if>
+      <dynamics damping="0.0" friction="0.0" />
+    </joint>
+    <link name="${prefix}arm_1_link">
+      <visual>
+        <geometry>
+        <xacro:unless value="${stl_mesh}">
+          <mesh filename="package://tm5_description/meshes/tm5_700/visual/tm5_700_arm1.obj" />
+        </xacro:unless>
+        <xacro:if value="${stl_mesh}">
+          <mesh filename="package://tm5_description/meshes/tm5_700/visual/tm5_700_arm1.stl" />
+        </xacro:if>
+        </geometry>
+        <material name="DarkOlive">
+          <color rgba="0.3 0.3 0.25 1.0" />
+        </material>
+      </visual>
+      <collision>
+        <geometry>
+          <mesh filename="package://tm5_description/meshes/tm5_700/collision/tm5_700_arm1_c.stl" />
+        </geometry>
+      </collision>
+      <xacro:cylinder_inertial_y radius="0.06" length="${arm_1_length}" mass="${arm_1_mass}">
+        <origin xyz="0 ${0.5*arm_1_length} 0" rpy="0 0 0" />
+      </xacro:cylinder_inertial_y>
+    </link>
+    <joint name="${prefix}elbow_joint" type="revolute">
       <parent link="${prefix}arm_1_link" />
       <child link = "${prefix}arm_2_link" />
-      <origin xyz="${arm_1_length} 0.0 ${elbow_offset}" rpy="0.0 0.0 0.0" />
-      <axis xyz="0 0 1" />
-      <xacro:unless value="${joint_limited}">
-        <limit lower="${-1.5 * pi}" upper="${1.5 * pi}" effort="150.0" velocity="3.15"/>
-      </xacro:unless>
-      <xacro:if value="${joint_limited}">
-        <limit lower="${-pi}" upper="${pi}" effort="150.0" velocity="3.15"/>
-      </xacro:if>
-      <dynamics damping="0.0" friction="0.0"/>
-    </joint>
-    <link name="${prefix}wrist_1_link">
-      <visual>
-        <geometry>
-	  <mesh filename="package://tm_description/meshes/tm700/visual/Wrist1.STL" />
-        </geometry>
-        <material name="DarkOlive">
-          <color rgba="0.3 0.3 0.25 1.0"/>
-        </material>
-      </visual>
-      <collision>
-        <geometry>
-	  <mesh filename="package://tm_description/meshes/tm700/collision/wrist_1.STL" />
-        </geometry>
-      </collision>
-      <xacro:cylinder_inertial radius="0.6" length="0.12" mass="${wrist_1_mass}">
-        <origin xyz="0.0 0.0 0.0" rpy="0 0 0" />
-      </xacro:cylinder_inertial>
+      <origin xyz="0 ${arm_1_length} ${-elbow_offset}" rpy="0 0 0" />
+      <axis xyz="0 0 -1" />
+      <limit lower="${elbow_lower_limit}" upper="${elbow_upper_limit}" effort="150.0" velocity="3.15" />
+      <xacro:if value="${safety_limits}">
+        <safety_controller soft_lower_limit="${elbow_lower_limit + safety_pos_margin}" soft_upper_limit="${elbow_upper_limit - safety_pos_margin}" k_position="${safety_k_position}" k_velocity="0.0"/>
+      </xacro:if>
+      <dynamics damping="0.0" friction="0.0" />
+    </joint>
+    <link name="${prefix}arm_2_link">
+      <visual>
+        <geometry>
+        <xacro:unless value="${stl_mesh}">
+          <mesh filename="package://tm5_description/meshes/tm5_700/visual/tm5_700_arm2.obj" />
+        </xacro:unless>
+        <xacro:if value="${stl_mesh}">
+          <mesh filename="package://tm5_description/meshes/tm5_700/visual/tm5_700_arm2.stl" />
+        </xacro:if>
+        </geometry>
+        <material name="DarkOlive">
+          <color rgba="0.3 0.3 0.25 1.0" />
+        </material>
+      </visual>
+      <collision>
+        <geometry>
+          <mesh filename="package://tm5_description/meshes/tm5_700/collision/tm5_700_arm2_c.stl" />
+        </geometry>
+      </collision>
+      <xacro:cylinder_inertial_y radius="0.045" length="${arm_2_length}" mass="${arm_2_mass}">
+        <origin xyz="0 ${0.5*arm_2_length} 0" rpy="0 0 0" />
+      </xacro:cylinder_inertial_y>
     </link>
     <joint name="${prefix}wrist_1_joint" type="revolute">
       <parent link="${prefix}arm_2_link" />
       <child link = "${prefix}wrist_1_link" />
-      <origin xyz="${arm_2_length} 0.0 ${wrist_offset}" rpy="${0.5 * pi} 0.0 ${0.5 * pi}" />
-      <axis xyz="0 1 0" />
-      <xacro:unless value="${joint_limited}">
-        <limit lower="${-2.0 * pi}" upper="${2.0 * pi}" effort="28.0" velocity="3.2"/>
-      </xacro:unless>
-      <xacro:if value="${joint_limited}">
-        <limit lower="${-pi}" upper="${pi}" effort="28.0" velocity="3.2"/>
-      </xacro:if>
-      <dynamics damping="0.0" friction="0.0"/>
-    </joint>
-    <link name="${prefix}wrist_2_link">
-      <visual>
-        <geometry>
-	  <mesh filename="package://tm_description/meshes/tm700/visual/Wrist2.STL" />
-        </geometry>
-        <material name="DarkOlive">
-          <color rgba="0.3 0.3 0.25 1.0"/>
-        </material>
-      </visual>
-      <collision>
-        <geometry>
-	  <mesh filename="package://tm_description/meshes/tm700/collision/wrist_2.STL" />
-        </geometry>
-      </collision>
-      <xacro:cylinder_inertial radius="0.6" length="0.12" mass="${wrist_2_mass}">
-        <origin xyz="0.0 0.0 0.0" rpy="0 0 0" />
-      </xacro:cylinder_inertial>
+      <origin xyz="0 ${arm_2_length} ${wrist_offset}" rpy="0 0 0" />
+      <axis xyz="0 0 -1" />
+      <limit lower="${wrist_1_lower_limit}" upper="${wrist_1_upper_limit}" effort="150.0" velocity="3.15"/>
+      <xacro:if value="${safety_limits}">
+        <safety_controller soft_lower_limit="${wrist_1_lower_limit + safety_pos_margin}" soft_upper_limit="${wrist_1_upper_limit - safety_pos_margin}" k_position="${safety_k_position}" k_velocity="0.0" />
+      </xacro:if>
+      <dynamics damping="0.0" friction="0.0" />
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
File: src/tmr_ros1/tm_description/urdf/tm700_robotique2f_robot_joint_limited.urdf.xacro (robot description, xacro)
@@ -1,12 +1,13 @@
 <?xml version="1.0"?>
-<robot name="tm700" xmlns:xacro="http://www.ros.org/wiki/xacro">
+<robot name="tm700_robotiq" xmlns:xacro="http://www.ros.org/wiki/xacro">
+  <xacro:arg name="transmission_hw_interface" default="hardware_interface/EffortJointInterface"/>
   <xacro:property name="prefix" value="" />
   <!-- gazebo stuff -->
   <xacro:include filename="$(find tm_description)/urdf/common.gazebo.xacro" />
-  <xacro:include filename="$(find tm_description)/urdf/tm.gazebo.xacro" />
+  <!-- <xacro:include filename="$(find tm_description)/urdf/tm.gazebo.xacro" /> -->
   <xacro:tm_arm_gazebo prefix="${prefix}" />
   <!-- tm700 -->
   <xacro:include filename="$(find tm_description)/urdf/tm700_robotique2f_gripper.urdf.xacro" />
-  <xacro:tm700_robot prefix="${prefix}" joint_limited="true" />
+  <xacro:tm700_robot prefix="${prefix}" joint_limited="true"  transmission_hw_interface="$(arg transmission_hw_interface)"/>
   <link name="world" />
   <joint name="world_joint" type="fixed">
