Commit message: new package tm5_700_grip_description

File: src/tmr_ros1/tm_description/urdf/tm700_robotique2f_robot_joint_limited_eih.urdf.xacro (robot description, xacro)
@@ -2,4 +2,5 @@
 <robot name="tm700_robotiq" xmlns:xacro="http://www.ros.org/wiki/xacro">
   <xacro:property name="prefix" value="" />
+  <xacro:arg name="transmission_hw_interface" default="hardware_interface/EffortJointInterface"/>
   <!-- gazebo stuff -->
   <xacro:include filename="$(find tm_description)/urdf/common.gazebo.xacro" />
@@ -8,5 +9,5 @@
   <!-- tm700 -->
   <xacro:include filename="$(find tm_description)/urdf/tm700_robotique2f_gripper.urdf.xacro" />
-  <xacro:tm700_robot prefix="${prefix}" joint_limited="true" />
+  <xacro:tm700_robot prefix="${prefix}" joint_limited="true" transmission_hw_interface="$(arg transmission_hw_interface)" />
   <link name="world" />
   <joint name="world_joint" type="fixed">

Commit message: fixed tm_gazebo tm700_gripper.launch (spawn model gazebo)

File: src/robotiq/robotiq_description/urdf/robotiq_85_gripper.transmission.xacro (robot description, xacro)
@@ -5,11 +5,11 @@
       <type>transmission_interface/SimpleTransmission</type>
       <joint name="${prefix}robotiq_85_left_knuckle_joint">
-        <hardwareInterface>PositionJointInterface</hardwareInterface>
-        <!-- <hardwareInterface>EffortJointInterface</hardwareInterface> -->
+        <!-- <hardwareInterface>PositionJointInterface</hardwareInterface> -->
+        <hardwareInterface>EffortJointInterface</hardwareInterface>
       </joint>
       <actuator name="${prefix}robotiq_85_left_knuckle_motor">
         <mechanicalReduction>1</mechanicalReduction>
-        <hardwareInterface>PositionJointInterface</hardwareInterface>
-        <!-- <hardwareInterface>EfforJointInterface</hardwareInterface> -->
+        <!-- <hardwareInterface>PositionJointInterface</hardwareInterface> -->
+        <hardwareInterface>EfforJointInterface</hardwareInterface>
       </actuator>
     </transmission>

File: src/tmr_ros1/tm5_700_gripper_description/urdf/tm700_robotiq_robot.urdf.xacro (robot description, xacro)
@@ -1,4 +1,4 @@
 <?xml version="1.0"?>
-<robot name="tm700_robotiq" xmlns:xacro="http://www.ros.org/wiki/xacro">
+<robot name="tm5_700_robotiq" xmlns:xacro="http://www.ros.org/wiki/xacro">
   <xacro:arg name="transmission_hw_interface" default="hardware_interface/PositionJointInterface" />
   <xacro:arg name="stl_mesh" default="false" />
@@ -7,11 +7,9 @@
   <!-- tm700 + 2f gripper -->
   <xacro:include filename="$(find tm5_700_gripper_description)/urdf/tm700_robotiq_gripper.urdf.xacro" />
-  <xacro:tm5_700_robotiq prefix="" joint_limited="false" stl_mesh="$(arg stl_mesh)"
-   transmission_hw_interface="$(arg transmission_hw_interface)" />
-  <link name="world" />
+  <!-- <link name="world" />
   <joint name="world_joint" type="fixed">
     <parent link="world" />
     <child link="base" />
     <origin xyz="0 0 0" rpy="0 0 0" />
-  </joint>
+  </joint> -->
 </robot>
