Commit message: adjusting tm_gazebo/launch/tm700.launch

File: src/tmr_ros1/tm5_700_gripper_description/urdf/tm5_700_robot.urdf.xacro (robot description, xacro)
@@ -2,4 +2,5 @@
 <robot xmlns:xacro="http://wiki.ros.org/xacro" name="tm5_700" >
   <!-- perche' NON FUNZIONA? <xacro:arg name="transmission_hw_interface" default="hardware_interface/PositionJointInterface" /> -->
+  <xacro:arg name="transmission_hw_interface" default="hardware_interface/PositionJointInterface" />
   <xacro:arg name="stl_mesh" default="false" />
   <!-- common stuff -->
@@ -8,5 +9,12 @@
   <xacro:include filename="$(find tm5_description)/urdf/tm5_700.urdf.xacro" />
   <!-- arm -->
-  <xacro:tm5_700_robot prefix="" joint_limited="false" stl_mesh="$(arg stl_mesh)" transmission_hw_interface="$(arg transmission_hw_interface)" />
+  <xacro:tm5_700_robot prefix="" joint_limited="false" stl_mesh="$(arg stl_mesh)"
+   shoulder_1_lower_limit="${-1.5*pi}"    shoulder_1_upper_limit="${1.5*pi}"
+   shoulder_2_lower_limit="${-pi}"        shoulder_2_upper_limit="${pi}"
+   elbow_lower_limit="${-pi}"             elbow_upper_limit="${pi}"
+   wrist_1_lower_limit="${-pi}"           wrist_1_upper_limit="${pi}"
+   wrist_2_lower_limit="${-pi}"           wrist_2_upper_limit="${pi}"
+   wrist_3_lower_limit="${-1.5*pi}"       wrist_3_upper_limit="${1.5*pi}"
+   transmission_hw_interface="$(arg transmission_hw_interface)" />
   <link name="world" />
   <joint name="world_joint" type="fixed">

File: src/tmr_ros1/tm5_700_gripper_description/urdf/tm700_robotiq_gripper.urdf.xacro (robot description, xacro)
@@ -1,4 +1,4 @@
 <?xml version="1.0"?>
-<robot name="tm700_robotiq" xmlns:xacro="http://www.ros.org/wiki/xacro">
+<robot name="tm5_700_robotiq" xmlns:xacro="http://www.ros.org/wiki/xacro">
   <xacro:include filename="$(find tm5_700_gripper_description)/urdf/tm5_700_robot.urdf.xacro" />
   <xacro:include filename="$(find robotiq_description)/urdf/robotiq_85_gripper.urdf.xacro" />

File: src/tmr_ros1/tm5_700_gripper_description/urdf/tm700_robotiq_robot.urdf.xacro (robot description, xacro)
@@ -1,14 +1,12 @@
 <?xml version="1.0"?>
 <robot name="tm700_robotiq" xmlns:xacro="http://www.ros.org/wiki/xacro">
-  <xacro:arg name="transmission_hw_interface" default="hardware_interface/EffortJointInterface" />
+  <xacro:arg name="transmission_hw_interface" default="hardware_interface/PositionJointInterface" />
   <xacro:arg name="stl_mesh" default="false" />
-  <xacro:property name="prefix" value="" />
   <!-- gazebo stuff -->
   <xacro:include filename="$(find tm5_description)/urdf/common.gazebo.xacro" />
-  <!-- <xacro:include filename="$(find tm5_description)/urdf/tm.gazebo.xacro" /> -->
-  <xacro:tm_arm_gazebo prefix="${prefix}" />
   <!-- tm700 + 2f gripper -->
   <xacro:include filename="$(find tm5_700_gripper_description)/urdf/tm700_robotiq_gripper.urdf.xacro" />
-  <xacro:tm5_700_robot prefix="${prefix}" joint_limited="false" stl_mesh="$(arg stl_mesh)" />
+  <xacro:tm5_700_robotiq prefix="" joint_limited="false" stl_mesh="$(arg stl_mesh)"
+   transmission_hw_interface="$(arg transmission_hw_interface)" />
   <link name="world" />
   <joint name="world_joint" type="fixed">

Commit message: ok

File: src/tmr_ros1/tm5_700_gripper_description/urdf/tm5_700_robot.urdf.xacro (robot description, xacro)
@@ -5,7 +5,7 @@
   <xacro:arg name="stl_mesh" default="false" />
   <!-- common stuff -->
-  <xacro:include filename="$(find tm5_description)/urdf/common.gazebo.xacro" />
+  <!--<xacro:include filename="$(find tm5_description)/urdf/common.gazebo.xacro" />-->
   <!-- tm5_700 -->
-  <xacro:include filename="$(find tm5_description)/urdf/tm5_700.urdf.xacro" />
+  <xacro:include filename="$(find tm5_700_gripper_description)/urdf/tm5_700.urdf.xacro" />
   <!-- arm -->
   <xacro:tm5_700_robot prefix="" joint_limited="false" stl_mesh="$(arg stl_mesh)"
@@ -17,9 +17,9 @@
    wrist_3_lower_limit="${-1.5*pi}"       wrist_3_upper_limit="${1.5*pi}"
    transmission_hw_interface="$(arg transmission_hw_interface)" />
-  <link name="world" />
+ <!--  <link name="world" />
   <joint name="world_joint" type="fixed">
     <parent link="world" />
     <child link="base" />
     <origin xyz="0 0 0" rpy="0 0 0" />
-  </joint>
+  </joint> -->
 </robot>

File: src/tmr_ros1/tm5_700_gripper_description/urdf/tm700_robotiq_robot.urdf.xacro (robot description, xacro)
@@ -7,9 +7,9 @@
   <!-- tm700 + 2f gripper -->
   <xacro:include filename="$(find tm5_700_gripper_description)/urdf/tm700_robotiq_gripper.urdf.xacro" />
-  <!-- <link name="world" />
+  <link name="world" />
   <joint name="world_joint" type="fixed">
     <parent link="world" />
     <child link="base" />
     <origin xyz="0 0 0" rpy="0 0 0" />
-  </joint> -->
+  </joint>
 </robot>
