Commit message: first_commit -> new tm5_700_gripper_moveit_config pkg

File: src/tmr_ros1/tm5_700_gripper_description/urdf/tm5_700.urdf.xacro (robot description, xacro)
@@ -313,6 +313,6 @@
     <link name="${prefix}base" />
     <joint name="${prefix}base-base_link" type="fixed">
-      <parent link="${prefix}base" />
-      <child link="${prefix}base_link" />
+      <parent link="${prefix}base_link" />
+      <child link="${prefix}base" />
       <origin xyz="0 0 0" rpy="${0.5 * pi} 0 0" /> <!-- Note: 0.5 * pi -->
     </joint>

File: src/tmr_ros1/tm5_700_gripper_description/urdf/tm5_700_robot.urdf.xacro (robot description, xacro)
@@ -1,12 +1,9 @@
 <?xml version="1.0"?>
 <robot xmlns:xacro="http://wiki.ros.org/xacro" name="tm5_700" >
-  <!-- perche' NON FUNZIONA? <xacro:arg name="transmission_hw_interface" default="hardware_interface/PositionJointInterface" /> -->
   <xacro:arg name="transmission_hw_interface" default="hardware_interface/PositionJointInterface" />
   <xacro:arg name="stl_mesh" default="false" />
-  <!-- common stuff -->
-  <!--<xacro:include filename="$(find tm5_description)/urdf/common.gazebo.xacro" />-->
   <!-- tm5_700 -->
   <xacro:include filename="$(find tm5_700_gripper_description)/urdf/tm5_700.urdf.xacro" />
-  <!-- arm -->
+  <!-- arm, joints limits is a required parameter-->
   <xacro:tm5_700_robot prefix="" joint_limited="false" stl_mesh="$(arg stl_mesh)"
    shoulder_1_lower_limit="${-1.5*pi}"    shoulder_1_upper_limit="${1.5*pi}"
@@ -17,9 +14,3 @@
    wrist_3_lower_limit="${-1.5*pi}"       wrist_3_upper_limit="${1.5*pi}"
    transmission_hw_interface="$(arg transmission_hw_interface)" />
- <!--  <link name="world" />
-  <joint name="world_joint" type="fixed">
-    <parent link="world" />
-    <child link="base" />
-    <origin xyz="0 0 0" rpy="0 0 0" />
-  </joint> -->
 </robot>

File: src/tmr_ros1/tm5_700_gripper_description/urdf/tm700_robotiq_gripper.urdf.xacro (robot description, xacro)
@@ -41,4 +41,11 @@
     <origin xyz="0 0 0.004" rpy="0 ${-pi/2} ${pi}"/>
   </xacro:robotiq_85_gripper>
+  <!-- define the tm5_700's position and orientation in the world coordinate system -->
+  <link name="world" />
+  <joint name="world_joint" type="fixed">
+    <parent link="world" />
+    <child link="base_link" /> <!-- TODO: check base_link name of robot -->
+    <origin xyz="0.0 0.0 0.0" rpy="${0.5 * pi} 0.0 0.0" />
+  </joint>
   <!-- Gazebo FT sensor plugin -->
   <gazebo reference="tool0">
