Commit message: Fixing TestTMclass.py and Tm5_700_boxes_scene.py for pick and place

File: src/tm5_700_gripper_simulation/demo_world/urdf/conveyor.urdf (robot description, URDF)
Before this commit: robot liukuhihna_gazebo, 3 links, 2 joints
Joints:
- joint fixed: origin xyz=0.0 0.0 0.0 rpy=0.0 0.0 0 -> xyz=0.0 1.0 0.0 rpy=0.0 0.0 0
