Commit message: adjusting urdf and config file for joints limits in position and velocity

File: src/tmr_ros1/tm12_description/urdf/tm12.urdf.xacro (robot description, xacro)
@@ -24,10 +24,10 @@
     shoulder_1_lower_limit:=${-1.5*pi}    shoulder_1_upper_limit:=${1.5*pi}
     shoulder_2_lower_limit:=${-pi}    shoulder_2_upper_limit:=${pi}
-    elbow_lower_limit:=${-pi}    elbow_upper_limit:=${pi}
+    elbow_lower_limit:=${-0.92*pi}    elbow_upper_limit:=${0.92*pi}
     wrist_1_lower_limit:=${-pi}    wrist_1_upper_limit:=${pi}
     wrist_2_lower_limit:=${-pi}    wrist_2_upper_limit:=${pi}
     wrist_3_lower_limit:=${-1.5*pi}    wrist_3_upper_limit:=${1.5*pi}
     transmission_hw_interface:=hardware_interface/PositionJointInterface
-    safety_limits:=false safety_pos_margin:=0.15
+    safety_limits:=true safety_pos_margin:=0.15
     safety_k_position:=20">
     <!-- Inertia parameters -->

File: src/tmr_ros1/tm12_description/urdf/tm12_palletizer.urdf.xacro (robot description, xacro)
@@ -8,5 +8,5 @@
   <!-- arm -->
   <!--xacro:tm12_robot prefix="" joint_limited="false" transmission_hw_interface="$(arg transmission_hw_interface)" /-->
-  <xacro:tm12_robot prefix="" joint_limited="false" stl_mesh="$(arg stl_mesh)" />
+  <xacro:tm12_robot prefix="" joint_limited="true" stl_mesh="$(arg stl_mesh)" />
     <!-- Joint to connect the gripper with the robot tool0 -->
     <joint name="gripper_joint" type="fixed">
@@ -21,6 +21,6 @@
           <mesh filename="package://tm12_description/meshes/tm12_1300/visual/schmalz_spb2.stl" />
         </geometry>
-        <material name="grey">
-          <color rgba="0.5 0.5 0.5 1"/>
+        <material name="light_blue">
+          <color rgba="0.3 1 1 1"/>
         </material>
       </visual>
@@ -41,5 +41,5 @@
       <parent link="world" />
       <child link="support" />
-      <origin xyz="0 0 0" rpy="0 0 0" />
+      <origin xyz="0 0 0.38" rpy="0 0 0" />
     </joint>
     <!-- Link that connect the robot with its cylindrical base-->
