Commit message: preparing file TestTMclass_tm12

File: src/palletizer_gazebo_simulation/demo_world/urdf/conveyor.urdf (robot description, URDF)
Before this commit: robot liukuhihna_gazebo, 3 links, 2 joints
Joints:
- removed joint fixed
- added joint fixed0: type fixed, parent world, child belt_visual, origin xyz=1.0 0.0 0.0 rpy=0.0 0.0 0

File: src/palletizer_gazebo_simulation/demo_world/urdf/red_cube.urdf (robot description, URDF)
Before this commit: robot red_cube, 1 links, 0 joints
Links:
- link base_link: mass 0.1 -> 0.3; geometry collision box size=0.30 0.21 0.165; visual box size=0.30 0.21 0.165
