Commit message: improving palletizer

File: src/palletizer_gazebo_simulation/demo_world/urdf/blue_slipsheet.urdf (robot description, URDF)
Before this commit: robot blue_cube, 1 links, 0 joints
Links:
- link base_link: geometry collision box size=0.505 0.675 0.015; visual box size=0.505 0.675 0.025

File: src/palletizer_gazebo_simulation/demo_world/urdf/conveyor.urdf (robot description, URDF)
Before this commit: robot liukuhihna_gazebo, 3 links, 2 joints
Joints:
- joint fixed0: origin xyz=1.0 0.0 0.0 rpy=0.0 0.0 0 -> xyz=1.07 0.0 0.0 rpy=0.0 0.0 0

File: src/palletizer_gazebo_simulation/demo_world/urdf/pallet1.urdf (robot description, URDF)
Before this commit: robot pallet1_gazebo, 2 links, 1 joints
Joints:
- joint fixed1: origin xyz=0.6 0.37 0.19 rpy=0.0 0.0 0 -> xyz=0.666 1.2 0.19 rpy=0.0 0.0 3.14

File: src/palletizer_gazebo_simulation/demo_world/urdf/red_cube.urdf (robot description, URDF)
Before this commit: robot red_cube, 1 links, 0 joints
Links:
- link base_link: mass 0.3 -> 0.1; geometry collision box size=0.305 0.215 0.157; visual box size=0.305 0.215 0.158

File: src/palletizer_gazebo_simulation/demo_world/urdf/sup_pallet1.urdf (robot description, URDF)
Before this commit: robot pallet2_gazebo, 2 links, 1 joints
Joints:
- joint fixed3: origin xyz=0.6 0.37 0 rpy=0.0 0.0 0 -> xyz=0.666 1.2 0.0 rpy=0.0 0.0 3.14

File: src/palletizer_gazebo_simulation/demo_world/urdf/sup_pallet2.urdf (robot description, URDF)
Before this commit: robot pallet2_gazebo, 2 links, 1 joints
Joints:
- joint fixed4: origin xyz=0.6 -1.15 0 rpy=0.0 0.0 0 -> xyz=-0.507 -1.1276 0 rpy=0.0 0.0 0

File: src/palletizer_gazebo_simulation/demo_world/urdf/sup_slipsheet.urdf (robot description, URDF)
Before this commit: robot pallet2_gazebo, 2 links, 1 joints
Links:
- removed link pallet_2
- added link sup_slipsheet, mass 40; collision mesh filename=package://demo_world/meshes/sup_slipsheet.stl; visual mesh filename=package://demo_world/meshes/sup_slipsheet.stl
Joints:
- removed joint fixed2
- added joint fixed1: type fixed, parent world, child sup_slipsheet, origin xyz=0.67 0.0 0.0 rpy=0.0 0.0 0.0

Commit message: gazebo_palletizer third demo

File: src/palletizer_gazebo_simulation/demo_world/urdf/blue_slipsheet.urdf (robot description, URDF)
Before this commit: robot blue_cube, 1 links, 0 joints
Links:
- link base_link: geometry collision box size=0.505 0.675 0.015; visual box size=0.505 0.675 0.015

File: src/palletizer_gazebo_simulation/demo_world/urdf/conveyor.urdf (robot description, URDF)
Before this commit: robot liukuhihna_gazebo, 3 links, 2 joints
Links:
- removed link belt_moving
Joints:
- removed joint belt_joint

File: src/palletizer_gazebo_simulation/demo_world/urdf/red_cube.urdf (robot description, URDF)
Before this commit: robot red_cube, 1 links, 0 joints
Links:
- link base_link: geometry collision box size=0.305 0.215 0.158; visual box size=0.305 0.215 0.158

File: src/palletizer_gazebo_simulation/demo_world/urdf/sup_slipsheet.urdf (robot description, URDF)
Before this commit: robot sup_slipsheets, 2 links, 1 joints
Joints:
- joint fixed1: origin xyz=0.67 0.0 0.0 rpy=0.0 0.0 0.0 -> xyz=0.55 0.04 0.0 rpy=0.0 0.0 0.0

File: src/tmr_ros1/tm12_description/urdf/tm12_palletizer.urdf.xacro (robot description, xacro)
@@ -36,4 +36,7 @@
       </inertial>
     </link>
+    <gazebo reference="vacuum_gripper">
+    <material>Gazebo/DarkGrey </material>
+  	</gazebo>
     <!-- Joint to connect the robot with the world frame -->
     <link name="world" />
@@ -60,4 +63,7 @@
       </inertial>
     </link>
+    <gazebo reference="support">
+    <material>Gazebo/Grey </material>
+  	</gazebo>
     <!-- Joint to connect the cylindrical base (support) with the base of the tm12_arm -->
     <joint name="sup_joint" type="fixed">
