Commit message: fixed palletizer pyshics version 1

File: src/palletizer_gazebo_simulation/demo_world/urdf/pallet1.urdf (robot description, URDF)
Before this commit: robot pallet1_gazebo, 2 links, 1 joints
Joints:
- joint fixed1: origin xyz=0.666 1.2 0.19 rpy=0.0 0.0 3.14 -> xyz=0.675 1.205 0.19 rpy=0.0 0.0 3.14

File: src/palletizer_gazebo_simulation/demo_world/urdf/sup_pallet1.urdf (robot description, URDF)
Before this commit: robot pallet2_gazebo, 2 links, 1 joints
Joints:
- joint fixed3: origin xyz=0.666 1.2 0.0 rpy=0.0 0.0 3.14 -> xyz=0.675 1.205 0.0 rpy=0.0 0.0 3.14
